Commit message: fixing kinematics for 5dof arm

File: mvp_arm_4dof_description/urdf/mvp_arm_4dof.xacro (robot description, xacro)
@@ -168,4 +168,5 @@
   <parent link="base_link"/>
   <child link="link_1_v1_1"/>
+	<limit effort="30" velocity="1.0" lower="-1.57" upper="1.57" />
   <axis xyz="-0.002854 0.005633 0.99998"/>
 </joint>
@@ -174,4 +175,5 @@
   <parent link="link_1_v1_1"/>
   <child link="link_2_v1_1"/>
+	<limit effort="30" velocity="1.0" lower="-1.57" upper="1.57" />
   <axis xyz="-0.025335 0.999663 -0.005703"/>
 </joint>
@@ -180,4 +182,5 @@
   <parent link="gripper_base_v1_1"/>
   <child link="gear2_v1_1"/>
+	<limit effort="30" velocity="1.0" lower="-1.57" upper="1.57" />
   <axis xyz="-0.141793 0.033815 0.989319"/>
 </joint>
@@ -186,4 +189,5 @@
   <parent link="gripper_base_v1_1"/>
   <child link="gear1_v1_1"/>
+	<limit effort="30" velocity="1.0" lower="-1.57" upper="1.57" />
   <axis xyz="-0.141793 0.033815 0.989319"/>
 </joint>
@@ -192,4 +196,5 @@
   <parent link="link_4_v1_1"/>
   <child link="gripper_base_v1_1"/>
+	<limit effort="30" velocity="1.0" lower="-1.57" upper="1.57" />
   <axis xyz="0.027296 -0.998903 0.038055"/>
 </joint>
@@ -203,4 +208,5 @@
   <parent link="link_2_v1_1"/>
   <child link="link_3_v1_1"/>
+	<limit effort="30" velocity="1.0" lower="-0.79" upper="0.79" />
   <axis xyz="0.025335 -0.999663 0.005703"/>
 </joint>
