Commit message: Added new gazebo world model, with new chessboard and chess pieces and updated kinematics with joint_state support and remade test_kinematics in python

File: arc_robot_arm/urdf/arm_with_camera.xacro (robot description, xacro)
@@ -6,5 +6,5 @@
 		<xacro:include filename="$(find realsense2_description)/urdf/_d435.urdf.xacro"/>
 		<xacro:sensor_d435 name="camera" topics_ns="camera" parent="gripper_base_v1_1" publish_pointcloud="true">
-			<origin xyz="0 0 0.02" rpy="0 0 ${pi}" />
+			<origin xyz="0 0 0.025" rpy="0 0.26 ${pi}" />
 		</xacro:sensor_d435>
 	</xacro:if>
