Commit message: descriptions added, moveit configs added, controllers work, plans work but does not execute due to trajectory time parameterization issue

File: protoarm_description/urdf/protoarm.xacro (robot description, xacro)
@@ -6,60 +6,179 @@
 <link name="world"/>
 <link name="base_link">
+	<inertial>
+    <origin xyz="0 0 0" rpy="0 0 0" />
+    <mass value="3.06" />
+    <inertia ixx="0.3" ixy="0.0" ixz="0.0" iyy="0.3" iyz="0.0" izz="0.3" />
+	</inertial>
+  <visual>
+    <origin rpy="0 0 0" xyz="0 0 0"/>
+    <geometry>
+      <mesh filename="package://protoarm_description/meshes/base_link.stl" scale="0.001 0.001 0.001"/>
+    </geometry>
+    <material name="silver_default"/>
+  </visual>
+  <collision>
+    <origin rpy="0 0 0" xyz="0 0 0"/>
+    <geometry>
+      <mesh filename="package://protoarm_description/meshes/base_link.stl" scale="0.001 0.001 0.001"/>
+    </geometry>
+  </collision>
+</link>
+<link name="shoulder_1">
+	<inertial>
+    <origin xyz="0 0 0" rpy="0 0 0" />
+    <mass value="3.06" />
+    <inertia ixx="0.3" ixy="0.0" ixz="0.0" iyy="0.3" iyz="0.0" izz="0.3" />
+	</inertial>
+  <visual>
+    <origin rpy="0 0 0" xyz="0.006279 -0.004346 -0.131179"/>
+    <geometry>
+      <mesh filename="package://protoarm_description/meshes/shoulder_1.stl" scale="0.001 0.001 0.001"/>
+    </geometry>
+    <material name="silver_default"/>
+  </visual>
+  <collision>
+    <origin rpy="0 0 0" xyz="0.006279 -0.004346 -0.131179"/>
+    <geometry>
+      <mesh filename="package://protoarm_description/meshes/shoulder_1.stl" scale="0.001 0.001 0.001"/>
+    </geometry>
+  </collision>
+</link>
+<link name="humerus_1">
+	<inertial>
+    <origin xyz="0 0 0" rpy="0 0 0" />
+    <mass value="3.06" />
+    <inertia ixx="0.3" ixy="0.0" ixz="0.0" iyy="0.3" iyz="0.0" izz="0.3" />
+	</inertial>
+  <visual>
+    <origin rpy="0 0 0" xyz="0.020207 -0.000222 -0.17144"/>
+    <geometry>
+      <mesh filename="package://protoarm_description/meshes/humerus_1.stl" scale="0.001 0.001 0.001"/>
+    </geometry>
+    <material name="silver_default"/>
+  </visual>
+  <collision>
+    <origin rpy="0 0 0" xyz="0.020207 -0.000222 -0.17144"/>
+    <geometry>
+      <mesh filename="package://protoarm_description/meshes/humerus_1.stl" scale="0.001 0.001 0.001"/>
+    </geometry>
+  </collision>
+</link>
+<link name="forearm_1">
+	<inertial>
+    <origin xyz="0 0 0" rpy="0 0 0" />
+    <mass value="3.06" />
+    <inertia ixx="0.3" ixy="0.0" ixz="0.0" iyy="0.3" iyz="0.0" izz="0.3" />
+	</inertial>
+  <visual>
+    <origin rpy="0 0 0" xyz="0.017319 -0.000979 -0.291403"/>
+    <geometry>
+      <mesh filename="package://protoarm_description/meshes/forearm_1.stl" scale="0.001 0.001 0.001"/>
+    </geometry>
+    <material name="silver_default"/>
+  </visual>
+  <collision>
+    <origin rpy="0 0 0" xyz="0.017319 -0.000979 -0.291403"/>
+    <geometry>
+      <mesh filename="package://protoarm_description/meshes/forearm_1.stl" scale="0.001 0.001 0.001"/>
+    </geometry>
+  </collision>
+</link>
+<link name="palm_1">
+	<inertial>
+    <origin xyz="0 0 0" rpy="0 0 0" />
+    <mass value="3.06" />
+    <inertia ixx="0.3" ixy="0.0" ixz="0.0" iyy="0.3" iyz="0.0" izz="0.3" />
+	</inertial>
+  <visual>
+    <origin rpy="0 0 0" xyz="0.135027 -0.00469 -0.297799"/>
+    <geometry>
+      <mesh filename="package://protoarm_description/meshes/palm_1.stl" scale="0.001 0.001 0.001"/>
+    </geometry>
+    <material name="silver_default"/>
+  </visual>
+  <collision>
+    <origin rpy="0 0 0" xyz="0.135027 -0.00469 -0.297799"/>
+    <geometry>
+      <mesh filename="package://protoarm_description/meshes/palm_1.stl" scale="0.001 0.001 0.001"/>
+    </geometry>
+  </collision>
+</link>
+<link name="right_finger_1">
+	<inertial>
+    <origin xyz="0 0 0" rpy="0 0 0" />
+    <mass value="0.05" />
+    <inertia ixx="0.1" ixy="0.0" ixz="0.0" iyy="0.1" iyz="0.0" izz="0.1" />
+	</inertial>
+  <visual>
+    <origin rpy="0 0 0" xyz="0.172286 -0.013294 -0.313884"/>
+    <geometry>
+      <mesh filename="package://protoarm_description/meshes/right_finger_1.stl" scale="0.001 0.001 0.001"/>
+    </geometry>
+    <material name="silver_default"/>
+  </visual>
+  <collision>
+    <origin rpy="0 0 0" xyz="0.172286 -0.013294 -0.313884"/>
+    <geometry>
+      <mesh filename="package://protoarm_description/meshes/right_finger_1.stl" scale="0.001 0.001 0.001"/>
+    </geometry>
+  </collision>
+</link>
+<link name="right_pad_1">
   <inertial>
     <origin xyz="0 0 0" rpy="0 0 0" />
-    <mass value="3.06" />
-    <inertia ixx="0.3" ixy="0.0" ixz="0.0" iyy="0.3" iyz="0.0" izz="0.3" />
-	</inertial>
-  <visual>
-    <origin rpy="0 0 0" xyz="0 0 0"/>
-    <geometry>
-      <mesh filename="package://protoarm_description/meshes/base_link.stl" scale="0.001 0.001 0.001"/>
-    </geometry>
-    <material name="silver_default"/>
-  </visual>
-  <collision>
-    <origin rpy="0 0 0" xyz="0 0 0"/>
-    <geometry>
-      <mesh filename="package://protoarm_description/meshes/base_link.stl" scale="0.001 0.001 0.001"/>
-    </geometry>
-  </collision>
-</link>
-<link name="shoulder_1">
+    <mass value="0.01"/>
+    <inertia ixx="0.0" ixy="0.0" ixz="-0.0" iyy="0.0" iyz="-0.0" izz="0.0"/>
+  </inertial>
+  <visual>
+    <origin rpy="0 0 0" xyz="0.221612 -0.041843 -0.322926"/>
+    <geometry>
+      <mesh filename="package://protoarm_description/meshes/right_pad_1.stl" scale="0.001 0.001 0.001"/>
+    </geometry>
+    <material name="silver_default"/>
+  </visual>
+  <collision>
+    <origin rpy="0 0 0" xyz="0.221612 -0.041843 -0.322926"/>
+    <geometry>
+      <mesh filename="package://protoarm_description/meshes/right_pad_1.stl" scale="0.001 0.001 0.001"/>
+    </geometry>
+  </collision>
+</link>
+<link name="left_finger_1">
+	<inertial>
+    <origin xyz="0 0 0" rpy="0 0 0" />
+    <mass value="0.05" />
+    <inertia ixx="0.1" ixy="0.0" ixz="0.0" iyy="0.1" iyz="0.0" izz="0.1" />
+	</inertial>
+  <visual>
+    <origin rpy="0 0 0" xyz="0.171552 0.013576 -0.314907"/>
+    <geometry>
+      <mesh filename="package://protoarm_description/meshes/left_finger_1.stl" scale="0.001 0.001 0.001"/>
+    </geometry>
+    <material name="silver_default"/>
+  </visual>
+  <collision>
+    <origin rpy="0 0 0" xyz="0.171552 0.013576 -0.314907"/>
+    <geometry>
+      <mesh filename="package://protoarm_description/meshes/left_finger_1.stl" scale="0.001 0.001 0.001"/>
+    </geometry>
+  </collision>
+</link>
+<link name="left_pad_1">
   <inertial>
     <origin xyz="0 0 0" rpy="0 0 0" />
-    <mass value="3.06" />
-    <inertia ixx="0.3" ixy="0.0" ixz="0.0" iyy="0.3" iyz="0.0" izz="0.3" />
-	</inertial>
-  <visual>
-    <origin rpy="0 0 0" xyz="0.006279 -0.004346 -0.131179"/>
-    <geometry>
-      <mesh filename="package://protoarm_description/meshes/shoulder_1.stl" scale="0.001 0.001 0.001"/>
-    </geometry>
-    <material name="silver_default"/>
-  </visual>
-  <collision>
-    <origin rpy="0 0 0" xyz="0.006279 -0.004346 -0.131179"/>
-    <geometry>
-      <mesh filename="package://protoarm_description/meshes/shoulder_1.stl" scale="0.001 0.001 0.001"/>
-    </geometry>
-  </collision>
-</link>
-<link name="humerus_1">
-  <inertial>
-    <origin xyz="0 0 0" rpy="0 0 0" />
-    <mass value="3.06" />
-    <inertia ixx="0.3" ixy="0.0" ixz="0.0" iyy="0.3" iyz="0.0" izz="0.3" />
-	</inertial>
-  <visual>
-    <origin rpy="0 0 0" xyz="0.020207 -0.000222 -0.17144"/>
-    <geometry>
-      <mesh filename="package://protoarm_description/meshes/humerus_1.stl" scale="0.001 0.001 0.001"/>
-    </geometry>
-    <material name="silver_default"/>
-  </visual>
-  <collision>
-    <origin rpy="0 0 0" xyz="0.020207 -0.000222 -0.17144"/>
-    <geometry>
-      <mesh filename="package://protoarm_description/meshes/humerus_1.stl" scale="0.001 0.001 0.001"/>
+    <mass value="0.01"/> <inertia ixx="0.0" ixy="0.0" ixz="-0.0" iyy="0.0" iyz="-0.0" izz="0.0"/>
+  </inertial>
+  <visual>
+    <origin rpy="0 0 0" xyz="0.221766 0.039676 -0.326185"/>
+    <geometry>
+      <mesh filename="package://protoarm_description/meshes/left_pad_1.stl" scale="0.001 0.001 0.001"/>
+    </geometry>
+    <material name="silver_default"/>
+  </visual>
+  <collision>
+    <origin rpy="0 0 0" xyz="0.221766 0.039676 -0.326185"/>
+    <geometry>
+      <mesh filename="package://protoarm_description/meshes/left_pad_1.stl" scale="0.001 0.001 0.001"/>
     </geometry>
   </collision>
@@ -67,8 +186,8 @@
 <link name="wrist_1">
   <inertial>
-    <origin xyz="0 0 0" rpy="0 0 0" />
-    <mass value="3.06" />
-    <inertia ixx="0.3" ixy="0.0" ixz="0.0" iyy="0.3" iyz="0.0" izz="0.3" />
-	</inertial>
+    <origin rpy="0 0 0" xyz="-0.017641925972066652 0.005015171425043511 0.005922235102376161"/>
+    <mass value="0.1295112121194818"/>
+    <inertia ixx="2e-05" ixy="4e-06" ixz="0.0" iyy="4e-05" iyz="-1e-06" izz="3.1e-05"/>
+  </inertial>
   <visual>
     <origin rpy="0 0 0" xyz="0.107006 0.008795 -0.291635"/>
@@ -82,124 +201,4 @@
     <geometry>
       <mesh filename="package://protoarm_description/meshes/wrist_1.stl" scale="0.001 0.001 0.001"/>
-    </geometry>
-  </collision>
-</link>
-<link name="forearm_1">
-  <inertial>
-    <origin xyz="0 0 0" rpy="0 0 0" />
-    <mass value="3.06" />
-    <inertia ixx="0.3" ixy="0.0" ixz="0.0" iyy="0.3" iyz="0.0" izz="0.3" />
-	</inertial>
-  <visual>
-    <origin rpy="0 0 0" xyz="0.017319 -0.000979 -0.291403"/>
-    <geometry>
-      <mesh filename="package://protoarm_description/meshes/forearm_1.stl" scale="0.001 0.001 0.001"/>
-    </geometry>
-    <material name="silver_default"/>
-  </visual>
-  <collision>
-    <origin rpy="0 0 0" xyz="0.017319 -0.000979 -0.291403"/>
-    <geometry>
-      <mesh filename="package://protoarm_description/meshes/forearm_1.stl" scale="0.001 0.001 0.001"/>
-    </geometry>
-  </collision>
-</link>
-<link name="palm_1">
-  <inertial>
-    <origin xyz="0 0 0" rpy="0 0 0" />
-    <mass value="3.06" />
-    <inertia ixx="0.3" ixy="0.0" ixz="0.0" iyy="0.3" iyz="0.0" izz="0.3" />
-	</inertial>
-  <visual>
-    <origin rpy="0 0 0" xyz="0.135027 -0.00469 -0.297799"/>
-    <geometry>
-      <mesh filename="package://protoarm_description/meshes/palm_1.stl" scale="0.001 0.001 0.001"/>
-    </geometry>
-    <material name="silver_default"/>
-  </visual>
-  <collision>
-    <origin rpy="0 0 0" xyz="0.135027 -0.00469 -0.297799"/>
-    <geometry>
-      <mesh filename="package://protoarm_description/meshes/palm_1.stl" scale="0.001 0.001 0.001"/>
-    </geometry>
-  </collision>
-</link>
-<link name="right_gear_1">
-  <inertial>
-    <origin xyz="0 0 0" rpy="0 0 0" />
-    <mass value="3.06" />
-    <inertia ixx="0.3" ixy="0.0" ixz="0.0" iyy="0.3" iyz="0.0" izz="0.3" />
-	</inertial>
-  <visual>
-    <origin rpy="0 0 0" xyz="0.172286 -0.013294 -0.313884"/>
-    <geometry>
-      <mesh filename="package://protoarm_description/meshes/right_gear_1.stl" scale="0.001 0.001 0.001"/>
-    </geometry>
-    <material name="silver_default"/>
-  </visual>
-  <collision>
-    <origin rpy="0 0 0" xyz="0.172286 -0.013294 -0.313884"/>
-    <geometry>
-      <mesh filename="package://protoarm_description/meshes/right_gear_1.stl" scale="0.001 0.001 0.001"/>
-    </geometry>
-  </collision>
-</link>
-<link name="right_finger_1">
-  <inertial>
-    <origin xyz="0 0 0" rpy="0 0 0"/>
-    <mass value="0.01"/>
-	  <inertia ixx="0.1" ixy="0.0" ixz="0.0" iyy="0.1" iyz="0.0" izz="0.1"/>
-  </inertial>
-  <visual>
-    <origin rpy="0 0 0" xyz="0.176409 -0.043875 -0.316941"/>
-    <geometry>
-      <mesh filename="package://protoarm_description/meshes/right_finger_1.stl" scale="0.001 0.001 0.001"/>
-    </geometry>
-    <material name="silver_default"/>
-  </visual>
-  <collision>
-    <origin rpy="0 0 0" xyz="0.176409 -0.043875 -0.316941"/>
-    <geometry>
-      <mesh filename="package://protoarm_description/meshes/right_finger_1.stl" scale="0.001 0.001 0.001"/>
-    </geometry>
-  </collision>
-</link>
-<link name="left_gear_1">
-  <inertial>
-    <origin xyz="0 0 0" rpy="0 0 0"/>
-    <mass value="0.01"/>
-	  <inertia ixx="0.1" ixy="0.0" ixz="0.0" iyy="0.1" iyz="0.0" izz="0.1"/>
-  </inertial>
-  <visual>
-    <origin rpy="0 0 0" xyz="0.171552 0.013576 -0.314907"/>
-    <geometry>
-      <mesh filename="package://protoarm_description/meshes/left_gear_1.stl" scale="0.001 0.001 0.001"/>
-    </geometry>
-    <material name="silver_default"/>
-  </visual>
-  <collision>
-    <origin rpy="0 0 0" xyz="0.171552 0.013576 -0.314907"/>
-    <geometry>
-      <mesh filename="package://protoarm_description/meshes/left_gear_1.stl" scale="0.001 0.001 0.001"/>
-    </geometry>
-  </collision>
-</link>
-<link name="left_finger_1">
-  <inertial>
-    <origin xyz="0 0 0" rpy="0 0 0"/>
-    <mass value="0.01"/>
-	  <inertia ixx="0.1" ixy="0.0" ixz="0.0" iyy="0.1" iyz="0.0" izz="0.1"/>
-  </inertial>
-  <visual>
-    <origin rpy="0 0 0" xyz="0.16646 0.043771 -0.319796"/>
-    <geometry>
-      <mesh filename="package://protoarm_description/meshes/left_finger_1.stl" scale="0.001 0.001 0.001"/>
-    </geometry>
-    <material name="silver_default"/>
-  </visual>
-  <collision>
-    <origin rpy="0 0 0" xyz="0.16646 0.043771 -0.319796"/>
-    <geometry>
-      <mesh filename="package://protoarm_description/meshes/left_finger_1.stl" scale="0.001 0.001 0.001"/>
     </geometry>
   </collision>
@@ -224,11 +223,4 @@
 </joint>
 <joint name="Rev3" type="continuous">
-  <origin rpy="0 0 0" xyz="-0.089687 -0.009774 0.000232"/>
-  <parent link="forearm_1"/>
-  <child link="wrist_1"/>
-  <axis xyz="-0.997823 -0.02494 0.061059"/>
-  <dynamics damping="1.0"/>
-</joint>
-<joint name="Rev4" type="continuous">
   <origin rpy="0 0 0" xyz="0.002888 0.000757 0.119963"/>
   <parent link="humerus_1"/>
@@ -244,31 +236,34 @@
   <dynamics damping="1.0"/>
 </joint>
-<joint name="G_Rev2" type="continuous">
+<joint name="G_Rev1" type="continuous">
   <origin rpy="0 0 0" xyz="-0.037259 0.008604 0.016085"/>
   <parent link="palm_1"/>
-  <child link="right_gear_1"/>
-  <axis xyz="0.063894 0.039735 0.997165"/>
-  <dynamics damping="1.0"/>
-</joint>
-<joint name="G_Rev3" type="continuous">
-  <origin rpy="0 0 0" xyz="-0.004123 0.030581 0.003057"/>
-  <parent link="right_gear_1"/>
   <child link="right_finger_1"/>
-  <axis xyz="0.063894 0.039735 0.997165"/>
-  <dynamics damping="1.0"/>
-</joint>
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
Commit message: gazebo sim + moveit control works

File: protoarm_description/urdf/protoarm.xacro (robot description, xacro)
@@ -108,5 +108,5 @@
 	<inertial>
     <origin xyz="0 0 0" rpy="0 0 0" />
-    <mass value="0.05" />
+    <mass value="0.1" />
     <inertia ixx="0.1" ixy="0.0" ixz="0.0" iyy="0.1" iyz="0.0" izz="0.1" />
 	</inertial>
@@ -126,9 +126,9 @@
 </link>
 <link name="right_pad_1">
-  <inertial>
-    <origin xyz="0 0 0" rpy="0 0 0" />
-    <mass value="0.01"/>
-    <inertia ixx="0.0" ixy="0.0" ixz="-0.0" iyy="0.0" iyz="-0.0" izz="0.0"/>
-  </inertial>
+	<inertial>
+    <origin xyz="0 0 0" rpy="0 0 0" />
+    <mass value="0.1" />
+    <inertia ixx="0.1" ixy="0.0" ixz="0.0" iyy="0.1" iyz="0.0" izz="0.1" />
+	</inertial>
   <visual>
     <origin rpy="0 0 0" xyz="0.221612 -0.041843 -0.322926"/>
@@ -148,5 +148,5 @@
 	<inertial>
     <origin xyz="0 0 0" rpy="0 0 0" />
-    <mass value="0.05" />
+    <mass value="0.1" />
     <inertia ixx="0.1" ixy="0.0" ixz="0.0" iyy="0.1" iyz="0.0" izz="0.1" />
 	</inertial>
@@ -166,8 +166,9 @@
 </link>
 <link name="left_pad_1">
-  <inertial>
-    <origin xyz="0 0 0" rpy="0 0 0" />
-    <mass value="0.01"/> <inertia ixx="0.0" ixy="0.0" ixz="-0.0" iyy="0.0" iyz="-0.0" izz="0.0"/>
-  </inertial>
+	<inertial>
+    <origin xyz="0 0 0" rpy="0 0 0" />
+    <mass value="0.1" />
+    <inertia ixx="0.1" ixy="0.0" ixz="0.0" iyy="0.1" iyz="0.0" izz="0.1" />
+	</inertial>
   <visual>
     <origin rpy="0 0 0" xyz="0.221766 0.039676 -0.326185"/>
