Commit message: added readmes, fixed launch files so they make sense and work, adjusted degree/position of realsense camera

File: protoarm_description/urdf/protoarm_realsense.xacro (robot description, xacro)
@@ -4,5 +4,5 @@
   <xacro:include filename="$(find realsense_ros_gazebo)/xacro/depthcam.xacro"/>
   <xacro:realsense_d435 sensor_name="camera" parent_link="forearm_1" rate="10">
-    <origin xyz="0 0.025 0.025" rpy="0 0.23 ${pi}" />
+    <origin xyz="-0.08 0 0.025" rpy="0 0 ${pi}" />
   </xacro:realsense_d435>
 </robot>
