Commit message: updated urdf

File: arm_description/urdf/arm.urdf.xacro (robot description, xacro)
@@ -152,6 +152,8 @@
       <parent link="link_4"/>
       <child link="link_5"/>
+      <axis xyz="0.0 0.0 1.0"/>
     </joint>
     <joint name="eef" type="fixed">
+      <origin rpy="0 0 0" xyz="0 0 $(arg J4_eef)"/>
       <parent link="link_5"/>
       <child link="eef"/>

Commit message: add camera tf

File: arm_description/urdf/arm.urdf.xacro (robot description, xacro)
@@ -119,4 +119,5 @@
     </link>
     <link name="eef"/>
+    <link name="overhead"/>
     <!-- revolute joints -->
     <joint name="joint_1" type="continuous">
@@ -154,4 +155,10 @@
       <axis xyz="0.0 0.0 1.0"/>
     </joint>
+    <joint name="arm_to_cam" type="fixed">
+      <origin rpy="0 0 0" xyz="-0.054 0 0.065"/>
+      <parent link="link_5"/>
+      <child link="overhead"/>
+      <axis xyz="0.0 0.0 1.0"/>
+    </joint>
     <joint name="eef" type="fixed">
       <origin rpy="0 0 0" xyz="0 0 $(arg J4_eef)"/>

Commit message: add keyboard control with RelaxedIK

File: arm_description/urdf/arm.urdf.xacro (robot description, xacro)
@@ -120,4 +120,5 @@
     <link name="eef"/>
     <link name="overhead"/>
+    <link name="chessboard"/>
     <!-- revolute joints -->
     <joint name="joint_1" type="continuous">
@@ -155,4 +156,11 @@
       <axis xyz="0.0 0.0 1.0"/>
     </joint>
+    <joint name="eef" type="fixed">
+      <origin rpy="0 0 0" xyz="0 0 $(arg J4_eef)"/>
+      <parent link="link_5"/>
+      <child link="eef"/>
+      <axis xyz="0.0 0.0 1.0"/>
+    </joint>
+    <!-- External transforms -->
     <joint name="arm_to_cam" type="fixed">
       <origin rpy="0 0 0" xyz="-0.054 0 0.065"/>
@@ -161,8 +169,8 @@
       <axis xyz="0.0 0.0 1.0"/>
     </joint>
-    <joint name="eef" type="fixed">
+    <joint name="" type="fixed">
       <origin rpy="0 0 0" xyz="0 0 $(arg J4_eef)"/>
-      <parent link="link_5"/>
-      <child link="eef"/>
+      <parent link="tag_2"/>
+      <child link="chessboard"/>
       <axis xyz="0.0 0.0 1.0"/>
     </joint>
